File: board-r3/teapot.kicad_pcb (KiCad board)
At the start: 2 copper layers, 29 x 57 mm, 51 parts, among them IC101 STM32F0xxCxUx, P1 BATT, P101 SMA, P3 SWD_TC, Q1 TEPT4400, U101 AMG88, U2 TLV61225, U4 RFM69W, U6 HTU21D, U7 MS5637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

Commit message: Convert r3 PCB to KiCAD v6 format
Other:
- net class Default removed
